File: boards/SET-1-Osiris-Avionics/SET_AV.kicad_pcb (KiCad board)
At the start: 2 copper layers, 64.5 x 85.5 mm, 31 parts, among them J1 ESP32P4ETH (header), J2 AP63203 Buck (header), J3 BMP388 (header), J4 LSM6DSOX (header), J5 XBee PRO S3B (header), J6 Adafruit PA1616D JST-XH heade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, J7 BR recovery signal, J8 BR staging signal

Commit message: SET 1 rev A complete
Parts:
- added C9: 100uF, Capacitor_SMD:C_1210_3225Metric_Pad1.33x2.70mm_HandSolder, F.Cu at (152.5, 70.6)
- added G***: RPL_Logo_NoSubtitle_15mm, rpl:RPL_Logo_NoSubtitle_15mm, F.Cu at (129.5, 66.5)
- added G***: RPL_Logo_26mm, rpl:RPL_Logo_26mm, B.Cu at (129.5, 65.1)
- added J10: Sensor Debug, Connector_PinHeader_2.54mm:PinHeader_1x08_P2.54mm_Vertical, F.Cu at (133.5, 113.9)
- added J11: Recovery Debug, rpl:PinHeader_1x03_P2.54mm_Vertical, F.Cu at (117.0, 104.5)
- added J12: Staging Debug, rpl:PinHeader_1x03_P2.54mm_Vertical, F.Cu at (116.5, 133.0)
- added J13: Battery Debug, rpl:PinHeader_1x03_P2.54mm_Vertical, F.Cu at (125.5, 112.5)
- added J14: GPS Debug, rpl:6-pin-debug, F.Cu at (124.0, 76.0)
- added J9: XBee Debug, rpl:6-pin-debug, F.Cu at (144.0, 65.9)
- BT1: renamed from + BAT -
- J1: value ESP32P4ETH (header) -> ESP32P4ETH (socket)
- J2: value AP63203 Buck (header) -> AP63203 Buck (socket)
- J3: value BMP388 (header) -> BMP388 (socket)
- J4: value LSM6DSOX (header) -> LSM6DSOX (socket)
- J5: value XBee PRO S3B (header) -> XBee PRO S3B (socket)
- moved C7 0.50 mm to (115.0, 68.0)
Routing:
- net /3V3: track 270.7 -> 291.1 mm
- net Net-(J1-22): track 7.63 -> 21.1 mm
- net Net-(J12-Pin_2): track 5.14 -> 16.4 mm
- net Net-(J11-Pin_2): track 5.01 -> 12.9 mm
- net Net-(J1-20): track 7.31 -> 13.8 mm
- net Net-(J14-Pin_3): track 28.9 -> 35.3 mm
- net Net-(J1-54): track 52.7 -> 58.8 mm
- net Net-(J1-19): track 59.4 -> 65.5 mm
- net Net-(J1-32): track 23.8 -> 29.4 mm
- net Net-(J1-18): track 52.4 -> 57.5 mm
- net Net-(J1-17): track 35.2 -> 40.2 mm
- net Net-(J1-15): track 36.5 -> 41.6 mm
- net Net-(J1-16): track 35.8 -> 40.9 mm
- net Net-(J1-6): track 50.8 -> 55.8 mm
- net Net-(J1-14): track 53.0 -> 58.0 mm
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Other:
- board text added: "Edgar was here"
- board text added: "Sophia Sanat Edgar Verastegui Medina Esha Rami Adel Afif Ayush Singhal Matthew Samonte Riley Parado Shirley Yu"
