File: boards/SET-1-Osiris-Avionics/SET_AV.kicad_sch (KiCad schematic)
At the start: 27 parts, among them J1 ESP32P4ETH (socket), J2 AP63203 Buck (socket), J3 BMP388 (socket), J4 LSM6DSOX (socket), J5 XBee PRO S3B (socket), J6 Adafruit PA1616D JST-XH heade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, J7 BR recovery signal, J8 BR staging signal

Commit message: SET 1 rev A complete
Parts:
- added C9: 100uF, Capacitor_SMD:C_1210_3225Metric_Pad1.33x2.70mm_HandSolder, symbol Device:C
- added J10: Sensor Debug, Connector_PinHeader_2.54mm:PinHeader_1x08_P2.54mm_Vertical, symbol Connector:Conn_01x08_Pin
- added J11: Recovery Debug, rpl:PinHeader_1x03_P2.54mm_Vertical, symbol Connector:Conn_01x03_Pin
- added J12: Staging Debug, rpl:PinHeader_1x03_P2.54mm_Vertical, symbol Connector:Conn_01x03_Pin
- added J13: Battery Debug, rpl:PinHeader_1x03_P2.54mm_Vertical, symbol Connector:Conn_01x03_Pin
- added J14: GPS Debug, rpl:6-pin-debug, symbol Connector:Conn_01x06_Pin
- added J9: XBee Debug, rpl:6-pin-debug, symbol Connector_Generic:Conn_01x06
- BT1: footprint TestPoint:TestPoint_2Pads_Pitch5.08mm_Drill1.3mm -> rpl:battery_pads; now not fitted
- C1, C5, C7: KiLib_Generator (none) -> capacitor/THT/other
- C2, C3, C4, C6, C8, R1, R10, R2, R3, R4, R5, R6, R7, R8, R9: KiLib_Generator (none) -> SMD_2terminal_chip_molded
- J6, J7, J8: KiLib_Generator (none) -> connector/JST
Connections:
- net 3V3: now also C9.1, J13.2 (Pin_2), J14.1 (Pin_1), J9.2 (Pin_2)
- net GND: now also C9.2, J11.3 (Pin_3), J12.3 (Pin_3), J13.1 (Pin_1), J14.6 (Pin_6), J9.5 (Pin_5)
- net at J1.31 (23), R8.1, R9.2: now also J11.1 (Pin_1)
- net at J8.2 (Pin_2), R6.1: now also J12.2 (Pin_2)
- net at J1.32 (22), R5.1, R6.2: now also J12.1 (Pin_1)
- net at C2.2, J1.35 (20), R3.1: now also J13.3 (Pin_3)
- net at J1.29 (26), J6.1 (PPS): now also J14.2 (Pin_2)
- net at J1.27, J6.4 (RX): now also J14.3 (Pin_3)
- net at J1.26 (32), J6.5 (TX): now also J14.4 (Pin_4)
- net at J1.25 (33), J6.6 (EN): now also J14.5 (Pin_5)
- net Net-(J1-4): now reaches J1.14 (3), J5.4 (DIN), R10.2
- net Net-(J1-4): now also J9.4 (Pin_4)
- net at J1.11 (5), J5.14 (CTS): now also J9.1 (Pin_1)
- net at J1.12 (4), J5.3 (DOUT): now also J9.3 (Pin_3)
- net at J1.15 (2), J5.6 (RST): now also J9.6 (Pin_6)
- net at J7.2 (Pin_2), R9.1: now also J11.2 (Pin_2)
- net at J1.1 (54), J3.4 (SCL), J4.4 (SCL): now also J10.8 (Pin_8)
- net at J1.2 (19), J3.6 (SDA), J4.5 (SDA): now also J10.7 (Pin_7)
- net at J1.4 (18), J3.5 (SDO), J4.6 (DO): now also J10.6 (Pin_6)
- net at J1.5 (17), J4.7 (CS): now also J10.5 (Pin_5)
- net at J1.6 (16), J4.8 (I1): now also J10.4 (Pin_4)
- net at J1.7 (15), J4.9 (I2): now also J10.3 (Pin_3)
- net at J1.10 (6), J3.8 (INT): now also J10.1 (Pin_1)
- net at J1.9 (14), J3.7 (CS): now also J10.2 (Pin_2)
